File: hardware/main_pcb/kicad_docs/analog_mux.sch (KiCad schematic (older format))
At the start: 1 part, among them U2 CD74HC4067SM

Commit message: progress on schemo
Parts:
- renumbered U2 to U6
Changed lines of the file:
@@
 S3
 $Comp
-L 74xx:CD74HC4067SM U2
+L 74xx:CD74HC4067SM U6
 U 1 1 5FB91F8F
 P 4050 3300
-F 0 "U2" H 4050 4481 50  0000 C CNN
+F 0 "U6" H 4050 4481 50  0000 C CNN
 F 1 "CD74HC4067SM" H 4050 4390 50  0000 C CNN
 F 2 "Package_SO:SSOP-24_5.3x8.2mm_P0.65mm" H 5100 2300 50  0001 C CIN
