File: hardware/main_pcb/kicad_docs/external_CV_scalers.sch (KiCad schematic (older format))
At the start: 3 parts, among them J14 CV_in_B, J15 CV_in_A, U7 MCP6002-xSN

Commit message: progress on schemo
Parts:
- renumbered J15 to J11, J14 to J12, U7 to U5
Changed lines of the file:
@@
 $EndDescr
 $Comp
-L Connector_Generic:Conn_01x03 J15
+L Connector_Generic:Conn_01x03 J11
 U 1 1 5FB8F3BE
 P 1300 1600
-F 0 "J15" H 1218 1917 50  0000 C CNN
+F 0 "J11" H 1218 1917 50  0000 C CNN
 F 1 "CV_in_A" H 1218 1826 50  0000 C CNN
 F 2 "Connector_PinHeader_2.54mm:PinHeader_1x03_P2.54mm_Vertical" H 1300 1600 50  0001 C CNN
@@
 $EndComp
 $Comp
-L Connector_Generic:Conn_01x03 J14
+L Connector_Generic:Conn_01x03 J12
 U 1 1 5FB8FB7F
 P 1250 2300
-F 0 "J14" H 1168 2617 50  0000 C CNN
+F 0 "J12" H 1168 2617 50  0000 C CNN
 F 1 "CV_in_B" H 1168 2526 50  0000 C CNN
 F 2 "Connector_PinHeader_2.54mm:PinHeader_1x03_P2.54mm_Vertical" H 1250 2300 50  0001 C CNN
@@
 $EndComp
 $Comp
-L Amplifier_Operational:MCP6002-xSN U7
+L Amplifier_Operational:MCP6002-xSN U5
 U 1 1 5FB98791
 P 4000 2250
-F 0 "U7" H 4000 2617 50  0000 C CNN
+F 0 "U5" H 4000 2617 50  0000 C CNN
 F 1 "MCP6002-xSN" H 4000 2526 50  0000 C CNN
 F 2 "Package_SO:SOIC-8_3.9x4.9mm_P1.27mm" H 4000 2250 50  0001 C CNN
@@
 $EndComp
 $Comp
-L Amplifier_Operational:MCP6002-xSN U7
+L Amplifier_Operational:MCP6002-xSN U5
 U 2 1 5FB99340
 P 4050 3600
-F 0 "U7" H 4050 3967 50  0000 C CNN
+F 0 "U5" H 4050 3967 50  0000 C CNN
 F 1 "MCP6002-xSN" H 4050 3876 50  0000 C CNN
 F 2 "Package_SO:SOIC-8_3.9x4.9mm_P1.27mm" H 4050 3600 50  0001 C CNN
