File: hardware/main_pcb/kicad_docs/microcontroller.sch (KiCad schematic (older format))
At the start: 1 part, among them U3 STM32G071KxT

Commit message: progress on schemo
Parts:
- renumbered U3 to U7
Changed lines of the file:
@@
 $EndDescr
 $Comp
-L MCU_ST_STM32G0:STM32G071KxT U3
+L MCU_ST_STM32G0:STM32G071KxT U7
 U 1 1 5FB948BE
 P 5500 3000
-F 0 "U3" H 5500 4281 50  0000 C CNN
+F 0 "U7" H 5500 4281 50  0000 C CNN
 F 1 "STM32G071KxT" H 5500 4190 50  0000 C CNN
 F 2 "Package_QFP:LQFP-32_7x7mm_P0.8mm" H 5400 1950 50  0001 R CNN
