File: hardware/main_pcb/kicad_docs/VCF_plug_in_board_ports.sch (KiCad schematic (older format))
At the start: 8 parts, among them J1 signal_in_A, J2 freq_CV_in_A, J3 signal_out_A, J4 feedback_CV_and_PS_A, J5 signal_in_B, J6 freq_CV_in_B, J7 signal_out_B, J8 feedback_CV_and_PS_B

Commit message: progress on pcb layout
Parts:
- renumbered J4 to J10, J5 to J11, J7 to J12, J6 to J13, J8 to J14, J1 to J7, J3 to J8, J2 to J9
Connections:
- net feedback_CV_in_A: now also J10.3 (Pin_3), J10.4 (Pin_4)
- net feedback_CV_in_B: now also J14.3 (Pin_3), J14.4 (Pin_4)
- net freq_CV_in_A: now also J9.3 (Pin_3), J9.4 (Pin_4)
- net freq_CV_in_B: now also J13.3 (Pin_3), J13.4 (Pin_4)
- net GND: now reaches J7.1 (Pin_1)
- net GND: now also J10.1 (Pin_1), J10.2 (Pin_2), J11.1 (Pin_1), J11.2 (Pin_2), J12.1 (Pin_1), J12.2 (Pin_2), J13.1 (Pin_1), J13.2 (Pin_2), J14.1 (Pin_1), J14.2 (Pin_2), J7.2 (Pin_2), J8.1 (Pin_1), J8.2 (Pin_2), J9.1 (Pin_1), J9.2 (Pin_2)
- net dry_in_A: now reaches J7.3 (Pin_3)
- net dry_in_A: now also J7.4 (Pin_4)
- net wet_out_A: now reaches J8.3 (Pin_3)
- net wet_out_A: now also J8.4 (Pin_4)
- net -12V: now reaches J10.5 (Pin_5)
- net -12V: now also J10.6 (Pin_6), J14.5 (Pin_5), J14.6 (Pin_6)
- net +12V: now reaches J10.7 (Pin_7)
- net +12V: now also J10.8 (Pin_8), J14.7 (Pin_7), J14.8 (Pin_8)
- net switched_in_B: now reaches J11.3 (Pin_3)
- net switched_in_B: now also J11.4 (Pin_4)
- net wet_out_B: now reaches J12.3 (Pin_3)
- net wet_out_B: now also J12.4 (Pin_4)
Other:
- note added: "VCF plug-in\nboard port A"
- note added: "VCF plug-in\nboard port B"
- moved on the sheet: J10, J11, J12, J13, J14, J7, J8, J9
