File: hardware/main_pcb/kicad_docs/control_voltage_generators.sch (KiCad schematic (older format))
At the start: 0 parts

Commit message: progress on pcb layout
Parts:
- added C28: 22n, Capacitor_SMD:C_0603_1608Metric, symbol Device:C
- added R20: 300k, Resistor_SMD:R_0603_1608Metric, symbol Device:R
- added R21: 120k, Resistor_SMD:R_0603_1608Metric, symbol Device:R
- added RV3: 10k, Potentiometer_THT:Potentiometer_Alpha_RD901F-40-00D_Single_Vertical, symbol Device:R_POT
- added U5: MCP6004, Package_SO:TSSOP-14_4.4x5mm_P0.65mm, symbol Amplifier_Operational:MCP6004
Connections:
- new net: C28.2, R20.1, R21.2, U5.2 (-)
- new net: R20.2, RV3.2
- new net -5V: RV3.3
- new net GND: RV3.1, U5.3 (+)
- new net feedback_cv_A: C28.1, R21.1, U5.1
Other:
- note added: "approx. range: \n[0v, +2v]"
- note added: "resonance CV generator"
