File: hardware/main_pcb/kicad_docs/lfo.sch (KiCad schematic (older format))
At the start: 21 parts, among them J15 swd_header, SW2 SW_SPDT_center_off, SW3 SW_SPDT, U10 STM32L031F4Px, U11 MCP4822

Commit message: reduce analog switch count, tidy up
Parts:
- renumbered U10 to U8, U11 to U9
Changed lines of the file:
@@
 $EndComp
 $Comp
-L Analog_DAC:MCP4822 U11
+L Analog_DAC:MCP4822 U9
 U 1 1 610932B4
 P 8950 3650
-F 0 "U11" H 8650 4200 50  0000 C CNN
+F 0 "U9" H 8650 4200 50  0000 C CNN
 F 1 "MCP4822" H 8650 4100 50  0000 C CNN
 F 2 "Package_SO:TSSOP-8_3x3mm_P0.65mm" H 9750 3350 50  0001 C CNN
@@
 lfo_inv_b_sw
 $Comp
-L MCU_ST_STM32L0:STM32L031F4Px U10
+L MCU_ST_STM32L0:STM32L031F4Px U8
 U 1 1 6111F64A
 P 6250 3850
-F 0 "U10" H 5800 4700 50  0000 C CNN
+F 0 "U8" H 5800 4700 50  0000 C CNN
 F 1 "STM32L031F4Px" H 5800 4550 50  0000 C CNN
 F 2 "Package_SO:TSSOP-20_4.4x6.5mm_P0.65mm" H 5850 3150 50  0001 R CNN
