File: hardware/main_pcb/kicad_docs/envelope_followers.sch (KiCad schematic (older format))
At the start: 2 parts, among them U5 MCP6002-xSN, U6 MCP6002-xSN

Commit message: progress on schemo
Parts:
- renumbered U5 to U3, U6 to U4
Changed lines of the file:
@@
 $EndDescr
 $Comp
-L Amplifier_Operational:MCP6002-xSN U5
+L Amplifier_Operational:MCP6002-xSN U3
 U 1 1 5FB93812
 P 2700 2400
-F 0 "U5" H 2700 2767 50  0000 C CNN
+F 0 "U3" H 2700 2767 50  0000 C CNN
 F 1 "MCP6002-xSN" H 2700 2676 50  0000 C CNN
 F 2 "Package_SO:SOIC-8_3.9x4.9mm_P1.27mm" H 2700 2400 50  0001 C CNN
@@
 $EndComp
 $Comp
-L Amplifier_Operational:MCP6002-xSN U5
+L Amplifier_Operational:MCP6002-xSN U3
 U 2 1 5FB948CB
 P 2750 3750
-F 0 "U5" H 2750 4117 50  0000 C CNN
+F 0 "U3" H 2750 4117 50  0000 C CNN
 F 1 "MCP6002-xSN" H 2750 4026 50  0000 C CNN
 F 2 "Package_SO:SOIC-8_3.9x4.9mm_P1.27mm" H 2750 3750 50  0001 C CNN
@@
 $EndComp
 $Comp
-L Amplifier_Operational:MCP6002-xSN U6
+L Amplifier_Operational:MCP6002-xSN U4
 U 1 1 5FB9583C
 P 5250 2400
-F 0 "U6" H 5250 2767 50  0000 C CNN
+F 0 "U4" H 5250 2767 50  0000 C CNN
 F 1 "MCP6002-xSN" H 5250 2676 50  0000 C CNN
 F 2 "Package_SO:SOIC-8_3.9x4.9mm_P1.27mm" H 5250 2400 50  0001 C CNN
@@
 $EndComp
 $Comp
-L Amplifier_Operational:MCP6002-xSN U6
+L Amplifier_Operational:MCP6002-xSN U4
 U 2 1 5FB96A17
 P 5300 3550
-F 0 "U6" H 5300 3917 50  0000 C CNN
+F 0 "U4" H 5300 3917 50  0000 C CNN
 F 1 "MCP6002-xSN" H 5300 3826 50  0000 C CNN
 F 2 "Package_SO:SOIC-8_3.9x4.9mm_P1.27mm" H 5300 3550 50  0001 C CNN

Commit message: progress on pcb layout
Parts:
- removed U3, U4: MCP6002-xSN, Package_SO:SOIC-8_3.9x4.9mm_P1.27mm, symbol Amplifier_Operational:MCP6002-xSN
- added C44, C45: 470n, Capacitor_SMD:C_0805_2012Metric, symbol Device:C
- added R43, R57: 20k, Resistor_SMD:R_0603_1608Metric, symbol Device:R
- added R44, R58: 10k, Resistor_SMD:R_0603_1608Metric, symbol Device:R
- added R45, R59: 30k, Resistor_SMD:R_0603_1608Metric, symbol Device:R
- added R46, R60: 4k7, Resistor_SMD:R_0603_1608Metric, symbol Device:R
- added R47, R61: 1k2, Resistor_SMD:R_0603_1608Metric, symbol Device:R
- added R48, R49, R50, R62, R63, R64: 100k, Resistor_SMD:R_0603_1608Metric, symbol Device:R
- added RV14, RV15: 100k trim, custom_footprints:bourns_3306F, symbol Device:R_POT
- added RV4: 500k_dual, Potentiometer_THT:Potentiometer_Alpha_RD902F-40-00D_Dual_Vertical, symbol Device:R_POT_Dual_Separate
- added RV5: 10k_dual, Potentiometer_THT:Potentiometer_Alpha_RD902F-40-00D_Dual_Vertical, symbol Device:R_POT_Dual_Separate
- added SW4: SW_DPDT_center_off, custom_footprints:DPDT_mini_toggle, symbol Switch:SW_DPDT_x2
- added U2, U3: MCP6004, Package_SO:TSSOP-14_4.4x5mm_P0.65mm, symbol Amplifier_Operational:MCP6004
Connections:
- new net: R44.1, R45.1, U2.5 (+)
- new net: R47.2, RV14.2, RV14.3, U2.6 (-)
- new net: R46.2, RV14.1, U2.7
- new net: R46.1, RV4.1
- new net: R43.1, R44.2, U2.2 (-)
- new net: C44.1, RV4.2, RV4.3, U2.10 (+)
- new net: R48.1, R50.2, U2.13 (-)
- new net: R48.2, R49.2, U2.8, U2.9 (-)
- new net: R49.1, SW4.2 (B), U2.12 (+)
- new net: R50.1, RV5.3, U2.14
- new net: R45.2, U2.1
- new net: C45.1, RV4.5, RV4.6, U3.10 (+)
- new net: R61.2, RV15.2, RV15.3, U3.6 (-)
- new net: R60.2, RV15.1, U3.7
- new net: R62.1, R64.2, U3.13 (-)
- new net: R62.2, R63.2, U3.8, U3.9 (-)
- new net: R63.1, SW4.5 (B), U3.12 (+)
- new net: R64.1, RV5.6, U3.14
- new net: R60.1, RV4.4
- new net: R59.2, U3.1
- new net: R57.1, R58.2, U3.2 (-)
- new net: R58.1, R59.1, U3.5 (+)
- new net +1V0: RV5.1, RV5.4, SW4.1 (A), SW4.3 (C), SW4.4 (A)
- new net GND: C44.2, C45.2, R47.1, R61.1, U2.3 (+), U3.3 (+)
- new net dry_A_in: R43.2
- new net dry_B_in: R57.2
- new net env_A: RV5.2
- new net env_B: RV5.5
- no-connect marks 0 -> 1
Other:
- note added: "Attack"
- note added: "approx. range: \n[0v, +2v]"
- note added: "check the orientation\nof the trimpots, try to\nmake it so they turn up\nand down intuitively"
- note added: "envelope A trim"
- note added: "envelope B trim"
- note added: "envelope mode switch:\n\nup-up\ndown-down\nup-down"
- note added: "envelope\nlevel"
- note added: "trim for approx.\nrange: [0v, +2v]"

Commit message: tidy up kicad docs
Other:
- note removed: "check the orientation\nof the trimpots, try to\nmake it so they turn up\nand down intuitively"
Changed lines of the file:
@@
 Wire Wire Line
 	7000 1750 7850 1750
-Text Notes 4450 3750 0    157  ~ 0
-check the orientation\nof the trimpots, try to\nmake it so they turn up\nand down intuitively
 $EndSCHEMATC
