File: hardware/main_pcb/kicad_docs/cv_summers.sch (KiCad schematic (older format))
At the start: 30 parts, among them U4 MCP6004

Commit message: tidy up kicad docs
Other:
- note added: "adjust such that +5v is developed\nacross an expression pedal connected\nvia the Tip-Ring-Sleeve jack."
- note removed: "check the orientation\nof the trimpots, try to\nmake it so they turn up\nand down intuitively"
Changed lines of the file:
@@
 Text Notes 4700 4500 0    79   ~ 0
 range: [0v, +2v]
-Text Notes 4700 3700 0    79   ~ 0
+Text Notes 4400 3700 0    79   ~ 0
 range: [-5v, 0v]
 Text Notes 6200 1250 0    79   ~ 0
@@
 	0    1    1    0
 $EndComp
-Text Notes 1850 6900 0    157  ~ 0
-check the orientation\nof the trimpots, try to\nmake it so they turn up\nand down intuitively
 Text Notes 8200 4550 0    157  ~ 0
 breadboard the scaler\ncircuits to make sure\nthere are no surprises
+Text Notes 1650 5100 0    50   ~ 0
+adjust such that +5v is developed\nacross an expression pedal connected\nvia the Tip-Ring-Sleeve jack.
+Text Notes 1700 6850 0    50   ~ 0
+adjust such that +5v is developed\nacross an expression pedal connected\nvia the Tip-Ring-Sleeve jack.
 $EndSCHEMATC

Commit message: tidy  up
Other:
- note removed: "breadboard the scaler\ncircuits to make sure\nthere are no surprises"
Changed lines of the file:
@@
 Wire Wire Line
 	6600 4500 6600 4900
-Text Label 6200 3700 2    50   ~ 0
+Text Label 5900 3700 2    50   ~ 0
 manual_freq
 $Comp
@@
 	0    1    1    0
 $EndComp
-Text Notes 8200 4550 0    157  ~ 0
-breadboard the scaler\ncircuits to make sure\nthere are no surprises
 Text Notes 1650 5100 0    50   ~ 0
 adjust such that +5v is developed\nacross an expression pedal connected\nvia the Tip-Ring-Sleeve jack.
 Text Notes 1700 6850 0    50   ~ 0
 adjust such that +5v is developed\nacross an expression pedal connected\nvia the Tip-Ring-Sleeve jack.
+Wire Wire Line
+	5900 3700 6200 3700
 $EndSCHEMATC
